File: hardware/IFB-40001-R02 - I2C_Encoder.brd (EAGLE design)
At the start: 20 x 30 mm, 32 parts, among them J3 CUTTABLE_JUMPER, J4 CUT_JUMPER_2X, U2 ATTINY841-MMHR

Commit message: updated hardware files
Parts:
- removed J1: (no value), SparkFun-Connectors:1X04_1MM_RA
- removed J3: CUTTABLE_JUMPER, PlayingWithFusion_Breakout-Lib:SMT_CUTTABLE_JUMPER
- added J5, J6: QWIICSIDE, PlayingWithFusion_JST:SM04B-SRSS-TB
- added R9: 100k, rcl:R0603
- J2: value (none) -> CUT_JUMPER_2X; device SparkFun-Connectors:1X04_1MM_RA -> PlayingWithFusion_Breakout-Lib:SMT_2X_CUTTABLE_JUMPER
- MT1: device PEC11R-4215F-S0024:XDCR_PEC11R-4215F-S0024 -> PlayingWithFusion_Bourns:XDCR_PEC11R-4215F-S0024
- moved J2 5.40 mm to (9.45, 10.9), turned to 180 degrees
- moved R1 2.45 mm to (3.96, 22.7), turned to 180 degrees
- moved C4 2.03 mm to (8.64, 19.9), turned to 180 degrees
- moved C3 1.36 mm to (8.64, 18.3), turned to 180 degrees
- moved R8 0.70 mm to (3.96, 19.3), turned to 180 degrees
- moved U$2 0.30 mm to (5.28, 27.2)
- moved C1 0.10 mm to (6.71, 10.1)
Connections:
- removed net ADDR: J3.2, R8.1, U2.12
- new net ADDR0: J2.3, R8.1, U2.12
- new net ADDR1: J2.1, R9.1, U2.11
- net GND: now also J2.2, J5.1, J6.1; no longer J1.1, J2.1, J3.1
- net SCL: now also J5.4, J6.4; no longer J1.4, J2.4
- net SDA: now also J5.3, J6.3; no longer J1.3, J2.3
- net VCC: now also J5.2, J6.2, R9.2; no longer J1.2, J2.2
Routing:
- net ADDR1: track 0.00 -> 15.3 mm, vias 0 -> 2
- net ADDR0: track 0.00 -> 12.9 mm
- net ADDR: track 9.45 -> 0.00 mm
- net SDA: track 33.6 -> 31.6 mm
- net PA1: track 13.7 -> 15.3 mm
- net GND: track 9.53 -> 8.12 mm
- net A: track 5.74 -> 6.61 mm
- net PA7: track 14.1 -> 13.3 mm
Other:
- board text added: "0 1"
- board text added: "R9"
