File: hardware/IFB-40001-R02 - I2C_Encoder.sch (EAGLE design)
At the start: 31 parts, among them J3 CUTTABLE_JUMPER, J4 CUT_JUMPER_2X, U2 ATTINY841-MMHR

Commit message: updated hardware files
Parts:
- removed J1: (no value), SparkFun-Connectors:QWIIC_CONNECTORJS-1MM
- removed J3: CUTTABLE_JUMPER, PlayingWithFusion_Breakout-Lib:CUTTABLE_JUMPER
- added J5, J6: QWIICSIDE, PlayingWithFusion_JST:QWIICSIDE
- added R9: 100k, rcl:R-US_R0603
- J2: value (none) -> CUT_JUMPER_2X; device SparkFun-Connectors:QWIIC_CONNECTORJS-1MM -> PlayingWithFusion_Breakout-Lib:CUT_JUMPER_2X
- MT1: device PEC11R-4215F-S0024:PEC11R-4215F-S0024 -> PlayingWithFusion_Bourns:PEC11R-4215F-S0024
Connections:
- removed net ADDR: J3.2, R8.1, U2.PB1
- new net ADDR0: J2.3, R8.1, U2.PB1
- new net ADDR1: J2.1, R9.1, U2.PB0
- net GND: now also J2.2, J5.1, J6.1; no longer J1.GND, J2.GND, J3.1
- net SCL: now also J5.4, J6.4; no longer J1.SCL, J2.SCL
- net SDA: now also J5.3, J6.3; no longer J1.SDA, J2.SDA
- net VCC: now also J5.2, J6.2, R9.2; no longer J1.VCC, J2.VCC
Other:
- moved on the sheet: R8
